File: KiCad/encoder.sch (KiCad schematic (older format))
At the start: 32 parts, among them P11 CONN_01X08, P12 ISP, P13 FTDI, P14 ENC_SS, SW1 ENC_RST, U5 ATMEGA328P, U6 3V3, X2 8MHz

Commit message: work in progress
Parts:
- C18, C19, C20, C21, C23, C24: footprint ArthurC Lib:c_0805 -> velokey-footprints:C_0603_HandSoldering
- C22, C25, C26, C27, C28: footprint ArthurC Lib:C_ELCO_SMD -> velokey-footprints:c_elec_3x5.3
- D6, D7: footprint ArthurC Lib:d_0805 -> velokey-footprints:C_0603
- P12: footprint ArthurC Lib:ISP -> velokey-footprints:Pin_Castellated_1x01
- P13: footprint ArthurC Lib:PIN_ARRAY-6X1 -> velokey-footprints:Pin_Castellated_1x01
- R12, R13, R14, R15, R16, R17, R18, R19, R20: footprint ArthurC Lib:r_0805 -> velokey-footprints:R_0603_HandSoldering
- SW1: footprint ArthurC Lib:SW_SMD -> velokey-footprints:SPST-PTS_810
- U5: footprint ArthurC Lib:TQFP32 -> SMD_Packages:PLCC-32
- U6: footprint ArthurC Lib:SOT23-3 -> velokey-footprints:TSOP-6
- X2: footprint ArthurC Lib:Xtal_SMD4 -> velokey-footprints:xtal_3.2x1.5mm
Changed lines of the file:
@@
 F 0 "C20" H 725 3250 40  0000 L CNB
 F 1 "22p" H 725 3175 40  0000 L CNN
-F 2 "ArthurC Lib:c_0805" H 700 3325 60  0001 C CNN
+F 2 "velokey-footprints:C_0603_HandSoldering" H 700 3325 60  0001 C CNN
 F 3 "" H 700 3325 60  0001 C CNN
 F 4 "mfr_pn" H 700 3325 60  0001 C CNN "manf#"
@@
 F 0 "C19" H 725 2850 40  0000 L CNB
 F 1 "22p" H 725 2925 40  0000 L CNN
-F 2 "ArthurC Lib:c_0805" H 700 2775 60  0001 C CNN
+F 2 "velokey-footprints:C_0603_HandSoldering" H 700 2775 60  0001 C CNN
 F 3 "" H 700 2775 60  0001 C CNN
 F 4 "mfr_pn" H 700 2775 60  0001 C CNN "manf#"
@@
 F 0 "C23" H 1675 7150 40  0000 L CNB
 F 1 "1uF" H 1675 7100 40  0000 L CNN
-F 2 "ArthurC Lib:c_0805" H 1600 7150 60  0001 C CNN
+F 2 "velokey-footprints:C_0603_HandSoldering" H 1600 7150 60  0001 C CNN
 F 3 "" H 1600 7150 60  0001 C CNN
 F 4 "mfr_pn" H 1600 7150 60  0001 C CNN "manf#"
@@
 F 0 "R16" H 6625 6750 40  0000 C CNB
 F 1 "750E" V 6525 6750 40  0000 C CNN
-F 2 "ArthurC Lib:r_0805" H 6525 6750 60  0001 C CNN
+F 2 "velokey-footprints:R_0603_HandSoldering" H 6525 6750 60  0001 C CNN
 F 3 "" H 6525 6750 60  0001 C CNN
 F 4 "mfr_pn" H 6525 6750 60  0001 C CNN "manf#"
@@
 F 0 "R15" H 6325 6750 40  0000 C CNB
 F 1 "750E" V 6225 6750 40  0000 C CNN
-F 2 "ArthurC Lib:r_0805" H 6225 6750 60  0001 C CNN
+F 2 "velokey-footprints:R_0603_HandSoldering" H 6225 6750 60  0001 C CNN
 F 3 "" H 6225 6750 60  0001 C CNN
 F 4 "mfr_pn" H 6225 6750 60  0001 C CNN "manf#"
@@
 F 0 "D7" V 6525 7350 40  0000 C CNB
 F 1 "LED" V 6625 7325 40  0000 C CNN
-F 2 "ArthurC Lib:d_0805" H 6525 7250 60  0001 C CNN
+F 2 "velokey-footprints:C_0603" H 6525 7250 60  0001 C CNN
 F 3 "" H 6525 7250 60  0001 C CNN
 	1    6525 7250
@@
 F 0 "D6" V 6225 7350 40  0000 C CNB
 F 1 "LED" V 6325 7325 40  0000 C CNN
-F 2 "ArthurC Lib:d_0805" H 6225 7250 60  0001 C CNN
+F 2 "velokey-footprints:C_0603" H 6225 7250 60  0001 C CNN
 F 3 "" H 6225 7250 60  0001 C CNN
 	1    6225 7250
@@
 F 0 "P12" V 3800 6800 40  0000 C CNB
 F 1 "ISP" V 3725 6800 40  0000 C CNN
-F 2 "ArthurC Lib:ISP" H 3725 7025 60  0001 C CNN
+F 2 "velokey-footprints:Pin_Castellated_1x01" H 3725 7025 60  0001 C CNN
 F 3 "" H 3725 7025 60  0001 C CNN
 F 4 "mfr_pn" H 3725 7025 60  0001 C CNN "manf#"
@@
 F 0 "C21" V 4900 6800 40  0000 C CNB
 F 1 "100n" V 4825 6800 40  0000 C CNN
-F 2 "ArthurC Lib:c_0805" H 5000 6800 60  0001 C CNN
+F 2 "velokey-footprints:C_0603_HandSoldering" H 5000 6800 60  0001 C CNN
 F 3 "" H 5000 6800 60  0001 C CNN
 F 4 "mfr_pn" H 5000 6800 60  0001 C CNN "manf#"
@@
 F 0 "P13" H 5500 6625 40  0000 C CNB
 F 1 "FTDI" H 5500 6700 40  0000 C CNN
-F 2 "ArthurC Lib:PIN_ARRAY-6X1" H 5500 7050 60  0001 C CNN
+F 2 "velokey-footprints:Pin_Castellated_1x01" H 5500 7050 60  0001 C CNN
 F 3 "" H 5500 7050 60  0001 C CNN
 F 4 "mfr_pn" H 5500 7050 60  0001 C CNN "manf#"
@@
 F 0 "U6" H 2075 6850 40  0000 C CNB
 F 1 "3V3" H 2375 6850 40  0000 C CNN
-F 2 "ArthurC Lib:SOT23-3" H 2225 7000 60  0001 C CNN
+F 2 "velokey-footprints:TSOP-6" H 2225 7000 60  0001 C CNN
 F 3 "" H 2225 7000 60  0001 C CNN
 F 4 "MCP1700T-3302E/TT" H 2225 7000 60  0001 C CNN "Part No"
@@
 F 0 "R14" H 4300 1550 40  0000 C CNB
 F 1 "10k" V 4250 1450 40  0000 C CNN
-F 2 "ArthurC Lib:r_0805" H 4250 1450 60  0001 C CNN
+F 2 "velokey-footprints:R_0603_HandSoldering" H 4250 1450 60  0001 C CNN
 F 3 "" H 4250 1450 60  0001 C CNN
 F 4 "mfr_pn" H 4250 1450 60  0001 C CNN "manf#"
@@
 F 0 "R13" H 4100 1550 40  0000 C CNB
 F 1 "10k" V 4050 1450 40  0000 C CNN
-F 2 "ArthurC Lib:r_0805" H 4050 1450 60  0001 C CNN
+F 2 "velokey-footprints:R_0603_HandSoldering" H 4050 1450 60  0001 C CNN
 F 3 "" H 4050 1450 60  0001 C CNN
 F 4 "mfr_pn" H 4050 1450 60  0001 C CNN "manf#"
@@
 F 0 "SW1" V 1075 4600 40  0000 C CNB
 F 1 "ENC_RST" V 975 4550 40  0000 C CNN
-F 2 "ArthurC Lib:SW_SMD" H 1075 4350 60  0001 C CNN
+F 2 "velokey-footprints:SPST-PTS_810" H 1075 4350 60  0001 C CNN
 F 3 "" H 1075 4350 60  0001 C CNN
 F 4 "mfr_pn" H 1075 4350 60  0001 C CNN "manf#"
@@
 F 0 "R12" H 1125 1550 40  0000 C CNB
 F 1 "10k" V 1075 1450 40  0000 C CNN
-F 2 "ArthurC Lib:r_0805" H 1075 1450 60  0001 C CNN
+F 2 "velokey-footprints:R_0603_HandSoldering" H 1075 1450 60  0001 C CNN
 F 3 "" H 1075 1450 60  0001 C CNN
 F 4 "mfr_pn" H 1075 1450 60  0001 C CNN "manf#"
@@
 F 0 "C18" H 1325 1450 40  0000 L CNB
 F 1 "100n" H 1325 1400 40  0000 L CNN
-F 2 "ArthurC Lib:c_0805" H 1250 1450 60  0001 C CNN
+F 2 "velokey-footprints:C_0603_HandSoldering" H 1250 1450 60  0001 C CNN
 F 3 "" H 1250 1450 60  0001 C CNN
 F 4 "mfr_pn" H 1250 1450 60  0001 C CNN "manf#"
@@
 F 0 "C24" H 2950 7150 40  0000 L CNB
 F 1 "1uF" H 2950 7100 40  0000 L CNN
-F 2 "ArthurC Lib:c_0805" H 2875 7150 60  0001 C CNN
+F 2 "velokey-footprints:C_0603_HandSoldering" H 2875 7150 60  0001 C CNN
 F 3 "" H 2875 7150 60  0001 C CNN
 F 4 "mfr_pn" H 2875 7150 60  0001 C CNN "manf#"
@@
 F 0 "U5" H 1700 4450 40  0000 L BNB
 F 1 "ATMEGA328P" H 1700 4375 40  0000 L BNN
-F 2 "ArthurC Lib:TQFP32" H 2925 1675 50  0001 C CNN
+F 2 "SMD_Packages:PLCC-32" H 2925 1675 50  0001 C CNN
 F 3 "" H 2400 3250 60  0001 C CNN
 F 4 "mfr_pn" H 2400 3250 60  0001 C CNN "manf#"
@@
 F 0 "X2" V 750 3100 40  0000 C CNB
 F 1 "8MHz" V 1050 3125 40  0000 C CNN
-F 2 "ArthurC Lib:Xtal_SMD4" H 900 3050 60  0001 C CNN
+F 2 "velokey-footprints:xtal_3.2x1.5mm" H 900 3050 60  0001 C CNN
 F 3 "" H 900 3050 60  0000 C CNN
 	1    900  3050
@@
 F 0 "C22" H 1300 7150 40  0000 L CNB
 F 1 "47uF,25V" H 1250 7075 40  0000 L CNN
-F 2 "ArthurC Lib:C_ELCO_SMD" H 1225 7150 60  0001 C CNN
+F 2 "velokey-footprints:c_elec_3x5.3" H 1225 7150 60  0001 C CNN
 F 3 "" H 1225 7150 60  0000 C CNN
 F 4 "mfr_pn" H 1225 7150 60  0001 C CNN "manf#"
@@
 F 0 "E1" H 6000 2225 40  0000 L CNB
 F 1 "ROT" H 6200 2225 40  0000 L CNN
-F 2 "" H 6150 1875 40  0000 C CNN
+F 2 "" H 6150 1875 40  0001 C CNN
 F 3 "" H 6150 1875 40  0000 C CNN
 F 4 "mfr_pn" H 6150 1875 40  0001 C CNN "manf#"
@@
 F 0 "E2" H 7675 2225 40  0000 L CNB
 F 1 "ROT" H 7875 2225 40  0000 L CNN
-F 2 "" H 7825 1875 40  0000 C CNN
+F 2 "" H 7825 1875 40  0001 C CNN
 F 3 "" H 7825 1875 40  0000 C CNN
 F 4 "mfr_pn" H 7825 1875 40  0001 C CNN "manf#"
@@
 F 0 "P11" H 4725 2975 40  0000 L CNB
 F 1 "CONN_01X08" V 4750 2450 40  0000 L CNB
-F 2 "" H 4650 2350 50  0000 C CNN
+F 2 "" H 4650 2350 50  0001 C CNN
 F 3 "" H 4650 2350 50  0000 C CNN
 	1    4650 2600
@@
 F 0 "P14" H 4200 4250 40  0000 L CNB
 F 1 "ENC_SS" H 4200 4225 40  0001 L CNB
-F 2 "" H 4125 4250 50  0000 C CNN
+F 2 "" H 4125 4250 50  0001 C CNN
 F 3 "" H 4125 4250 50  0000 C CNN
 	1    4125 4250
@@
 F 0 "C25" H 5975 2550 40  0000 L CNB
 F 1 "1uF" H 5925 2475 40  0000 L CNN
-F 2 "ArthurC Lib:C_ELCO_SMD" H 5900 2550 60  0001 C CNN
+F 2 "velokey-footprints:c_elec_3x5.3" H 5900 2550 60  0001 C CNN
 F 3 "" H 5900 2550 60  0000 C CNN
 F 4 "mfr_pn" H 5900 2550 60  0001 C CNN "manf#"
@@
 F 0 "C26" H 6475 2550 40  0000 L CNB
 F 1 "1uF" H 6425 2475 40  0000 L CNN
-F 2 "ArthurC Lib:C_ELCO_SMD" H 6400 2550 60  0001 C CNN
+F 2 "velokey-footprints:c_elec_3x5.3" H 6400 2550 60  0001 C CNN
 F 3 "" H 6400 2550 60  0000 C CNN
 F 4 "mfr_pn" H 6400 2550 60  0001 C CNN "manf#"
@@
 F 0 "C27" H 7650 2550 40  0000 L CNB
 F 1 "1uF" H 7600 2475 40  0000 L CNN
-F 2 "ArthurC Lib:C_ELCO_SMD" H 7575 2550 60  0001 C CNN
+F 2 "velokey-footprints:c_elec_3x5.3" H 7575 2550 60  0001 C CNN
 F 3 "" H 7575 2550 60  0000 C CNN
 F 4 "mfr_pn" H 7575 2550 60  0001 C CNN "manf#"
@@
 F 0 "C28" H 8150 2550 40  0000 L CNB
 F 1 "1uF" H 8100 2475 40  0000 L CNN
-F 2 "ArthurC Lib:C_ELCO_SMD" H 8075 2550 60  0001 C CNN
+F 2 "velokey-footprints:c_elec_3x5.3" H 8075 2550 60  0001 C CNN
 F 3 "" H 8075 2550 60  0000 C CNN
 F 4 "mfr_pn" H 8075 2550 60  0001 C CNN "manf#"
@@
 F 0 "R17" H 5950 2350 40  0000 C CNB
 F 1 "10k" V 5900 2250 40  0000 C CNN
-F 2 "ArthurC Lib:r_0805" H 5900 2250 60  0001 C CNN
+F 2 "velokey-footprints:R_0603_HandSoldering" H 5900 2250 60  0001 C CNN
 F 3 "" H 5900 2250 60  0001 C CNN
 F 4 "mfr_pn" H 5900 2250 60  0001 C CNN "manf#"
@@
 F 0 "R18" H 6450 2350 40  0000 C CNB
 F 1 "10k" V 6400 2250 40  0000 C CNN
-F 2 "ArthurC Lib:r_0805" H 6400 2250 60  0001 C CNN
+F 2 "velokey-footprints:R_0603_HandSoldering" H 6400 2250 60  0001 C CNN
 F 3 "" H 6400 2250 60  0001 C CNN
 F 4 "mfr_pn" H 6400 2250 60  0001 C CNN "manf#"
@@
 F 0 "R19" H 7625 2350 40  0000 C CNB
 F 1 "10k" V 7575 2250 40  0000 C CNN
-F 2 "ArthurC Lib:r_0805" H 7575 2250 60  0001 C CNN
+F 2 "velokey-footprints:R_0603_HandSoldering" H 7575 2250 60  0001 C CNN
 F 3 "" H 7575 2250 60  0001 C CNN
 F 4 "mfr_pn" H 7575 2250 60  0001 C CNN "manf#"
@@
 F 0 "R20" H 8125 2350 40  0000 C CNB
 F 1 "10k" V 8075 2250 40  0000 C CNN
-F 2 "ArthurC Lib:r_0805" H 8075 2250 60  0001 C CNN
+F 2 "velokey-footprints:R_0603_HandSoldering" H 8075 2250 60  0001 C CNN
 F 3 "" H 8075 2250 60  0001 C CNN
 F 4 "mfr_pn" H 8075 2250 60  0001 C CNN "manf#"

Commit message: added OTS schematic
Parts:
- C18, C21, C23, C24: footprint velokey-footprints:C_0603_HandSoldering -> (none); manf# mfr_pn -> (none)
- C19, C20: footprint velokey-footprints:C_0603_HandSoldering -> (none); Digikey 490-1734-1-ND -> (none); manf# mfr_pn -> (none)
- C22, C25, C26, C27, C28: footprint velokey-footprints:c_elec_3x5.3 -> (none); manf# mfr_pn -> (none)
- D6, D7: footprint velokey-footprints:C_0603 -> (none)
- E1, E2: manf# mfr_pn -> (none)
- P12, P13: footprint velokey-footprints:Pin_Castellated_1x01 -> (none); manf# mfr_pn -> (none)
- R12, R13, R14, R15, R16, R17, R18, R19, R20: footprint velokey-footprints:R_0603_HandSoldering -> (none); manf# mfr_pn -> (none)
- SW1: footprint velokey-footprints:SPST-PTS_810 -> (none); manf# mfr_pn -> (none)
- U5: footprint SMD_Packages:PLCC-32 -> (none); manf# mfr_pn -> (none)
- U6: footprint velokey-footprints:TSOP-6 -> (none); Part No MCP1700T-3302E/TT -> (none)
- X2: footprint velokey-footprints:xtal_3.2x1.5mm -> (none)
Changed lines of the file:
@@
 F 0 "C20" H 725 3250 40  0000 L CNB
 F 1 "22p" H 725 3175 40  0000 L CNN
-F 2 "velokey-footprints:C_0603_HandSoldering" H 700 3325 60  0001 C CNN
+F 2 "" H 700 3325 60  0001 C CNN
 F 3 "" H 700 3325 60  0001 C CNN
-F 4 "mfr_pn" H 700 3325 60  0001 C CNN "manf#"
-F 5 "490-1734-1-ND" H 700 3525 60  0001 C CNN "Digikey"
+F 4 "" H 700 3325 60  0001 C CNN "manf#"
 	1    700  3325
 	1    0    0    -1
@@
 F 0 "C19" H 725 2850 40  0000 L CNB
 F 1 "22p" H 725 2925 40  0000 L CNN
-F 2 "velokey-footprints:C_0603_HandSoldering" H 700 2775 60  0001 C CNN
+F 2 "" H 700 2775 60  0001 C CNN
 F 3 "" H 700 2775 60  0001 C CNN
-F 4 "mfr_pn" H 700 2775 60  0001 C CNN "manf#"
-F 5 "490-1734-1-ND" H 700 2975 60  0001 C CNN "Digikey"
+F 4 "" H 700 2775 60  0001 C CNN "manf#"
 	1    700  2775
 	1    0    0    -1
@@
 F 0 "C23" H 1675 7150 40  0000 L CNB
 F 1 "1uF" H 1675 7100 40  0000 L CNN
-F 2 "velokey-footprints:C_0603_HandSoldering" H 1600 7150 60  0001 C CNN
+F 2 "" H 1600 7150 60  0001 C CNN
 F 3 "" H 1600 7150 60  0001 C CNN
-F 4 "mfr_pn" H 1600 7150 60  0001 C CNN "manf#"
+F 4 "" H 1600 7150 60  0001 C CNN "manf#"
 	1    1600 7150
 	1    0    0    -1
@@
 F 0 "R16" H 6625 6750 40  0000 C CNB
 F 1 "750E" V 6525 6750 40  0000 C CNN
-F 2 "velokey-footprints:R_0603_HandSoldering" H 6525 6750 60  0001 C CNN
+F 2 "" H 6525 6750 60  0001 C CNN
 F 3 "" H 6525 6750 60  0001 C CNN
-F 4 "mfr_pn" H 6525 6750 60  0001 C CNN "manf#"
+F 4 "" H 6525 6750 60  0001 C CNN "manf#"
 	1    6525 6750
 	1    0    0    -1
@@
 F 0 "R15" H 6325 6750 40  0000 C CNB
 F 1 "750E" V 6225 6750 40  0000 C CNN
-F 2 "velokey-footprints:R_0603_HandSoldering" H 6225 6750 60  0001 C CNN
+F 2 "" H 6225 6750 60  0001 C CNN
 F 3 "" H 6225 6750 60  0001 C CNN
-F 4 "mfr_pn" H 6225 6750 60  0001 C CNN "manf#"
+F 4 "" H 6225 6750 60  0001 C CNN "manf#"
 	1    6225 6750
 	1    0    0    -1
@@
 F 0 "D7" V 6525 7350 40  0000 C CNB
 F 1 "LED" V 6625 7325 40  0000 C CNN
-F 2 "velokey-footprints:C_0603" H 6525 7250 60  0001 C CNN
+F 2 "" H 6525 7250 60  0001 C CNN
 F 3 "" H 6525 7250 60  0001 C CNN
 	1    6525 7250
@@
 F 0 "D6" V 6225 7350 40  0000 C CNB
 F 1 "LED" V 6325 7325 40  0000 C CNN
-F 2 "velokey-footprints:C_0603" H 6225 7250 60  0001 C CNN
+F 2 "" H 6225 7250 60  0001 C CNN
 F 3 "" H 6225 7250 60  0001 C CNN
 	1    6225 7250
@@
 F 0 "P12" V 3800 6800 40  0000 C CNB
 F 1 "ISP" V 3725 6800 40  0000 C CNN
-F 2 "velokey-footprints:Pin_Castellated_1x01" H 3725 7025 60  0001 C CNN
+F 2 "" H 3725 7025 60  0001 C CNN
 F 3 "" H 3725 7025 60  0001 C CNN
-F 4 "mfr_pn" H 3725 7025 60  0001 C CNN "manf#"
+F 4 "" H 3725 7025 60  0001 C CNN "manf#"
 	1    3725 7025
 	0    -1   -1   0
@@
 F 0 "C21" V 4900 6800 40  0000 C CNB
 F 1 "100n" V 4825 6800 40  0000 C CNN
-F 2 "velokey-footprints:C_0603_HandSoldering" H 5000 6800 60  0001 C CNN
+F 2 "" H 5000 6800 60  0001 C CNN
 F 3 "" H 5000 6800 60  0001 C CNN
-F 4 "mfr_pn" H 5000 6800 60  0001 C CNN "manf#"
+F 4 "" H 5000 6800 60  0001 C CNN "manf#"
 	1    5000 6800
 	0    1    1    0
@@
 F 0 "P13" H 5500 6625 40  0000 C CNB
 F 1 "FTDI" H 5500 6700 40  0000 C CNN
-F 2 "velokey-footprints:Pin_Castellated_1x01" H 5500 7050 60  0001 C CNN
+F 2 "" H 5500 7050 60  0001 C CNN
 F 3 "" H 5500 7050 60  0001 C CNN
-F 4 "mfr_pn" H 5500 7050 60  0001 C CNN "manf#"
+F 4 "" H 5500 7050 60  0001 C CNN "manf#"
 	1    5500 7050
 	1    0    0    1
@@
 F 0 "U6" H 2075 6850 40  0000 C CNB
 F 1 "3V3" H 2375 6850 40  0000 C CNN
-F 2 "velokey-footprints:TSOP-6" H 2225 7000 60  0001 C CNN
+F 2 "" H 2225 7000 60  0001 C CNN
 F 3 "" H 2225 7000 60  0001 C CNN
-F 4 "MCP1700T-3302E/TT" H 2225 7000 60  0001 C CNN "Part No"
+F 4 "" H 2225 7000 60  0001 C CNN "manf#"
 	1    2225 7000
 	1    0    0    -1
@@
 F 0 "R14" H 4300 1550 40  0000 C CNB
 F 1 "10k" V 4250 1450 40  0000 C CNN
-F 2 "velokey-footprints:R_0603_HandSoldering" H 4250 1450 60  0001 C CNN
+F 2 "" H 4250 1450 60  0001 C CNN
 F 3 "" H 4250 1450 60  0001 C CNN
-F 4 "mfr_pn" H 4250 1450 60  0001 C CNN "manf#"
+F 4 "" H 4250 1450 60  0001 C CNN "manf#"
 	1    4250 1450
 	1    0    0    -1
@@
 F 0 "R13" H 4100 1550 40  0000 C CNB
 F 1 "10k" V 4050 1450 40  0000 C CNN
-F 2 "velokey-footprints:R_0603_HandSoldering" H 4050 1450 60  0001 C CNN
+F 2 "" H 4050 1450 60  0001 C CNN
 F 3 "" H 4050 1450 60  0001 C CNN
-F 4 "mfr_pn" H 4050 1450 60  0001 C CNN "manf#"
+F 4 "" H 4050 1450 60  0001 C CNN "manf#"
 	1    4050 1450
 	1    0    0    -1
@@
 F 0 "SW1" V 1075 4600 40  0000 C CNB
 F 1 "ENC_RST" V 975 4550 40  0000 C CNN
-F 2 "velokey-footprints:SPST-PTS_810" H 1075 4350 60  0001 C CNN
+F 2 "" H 1075 4350 60  0001 C CNN
 F 3 "" H 1075 4350 60  0001 C CNN
-F 4 "mfr_pn" H 1075 4350 60  0001 C CNN "manf#"
+F 4 "" H 1075 4350 60  0001 C CNN "manf#"
 	1    1075 4350
 	0    -1   -1   0
@@
 F 0 "R12" H 1125 1550 40  0000 C CNB
 F 1 "10k" V 1075 1450 40  0000 C CNN
-F 2 "velokey-footprints:R_0603_HandSoldering" H 1075 1450 60  0001 C CNN
+F 2 "" H 1075 1450 60  0001 C CNN
 F 3 "" H 1075 1450 60  0001 C CNN
-F 4 "mfr_pn" H 1075 1450 60  0001 C CNN "manf#"
+F 4 "" H 1075 1450 60  0001 C CNN "manf#"
 	1    1075 1450
 	1    0    0    -1
@@
 F 0 "C18" H 1325 1450 40  0000 L CNB
 F 1 "100n" H 1325 1400 40  0000 L CNN
-F 2 "velokey-footprints:C_0603_HandSoldering" H 1250 1450 60  0001 C CNN
+F 2 "" H 1250 1450 60  0001 C CNN
 F 3 "" H 1250 1450 60  0001 C CNN
-F 4 "mfr_pn" H 1250 1450 60  0001 C CNN "manf#"
+F 4 "" H 1250 1450 60  0001 C CNN "manf#"
 	1    1250 1450
 	1    0    0    -1
@@
 F 0 "C24" H 2950 7150 40  0000 L CNB
 F 1 "1uF" H 2950 7100 40  0000 L CNN
-F 2 "velokey-footprints:C_0603_HandSoldering" H 2875 7150 60  0001 C CNN
+F 2 "" H 2875 7150 60  0001 C CNN
 F 3 "" H 2875 7150 60  0001 C CNN
-F 4 "mfr_pn" H 2875 7150 60  0001 C CNN "manf#"
+F 4 "" H 2875 7150 60  0001 C CNN "manf#"
 	1    2875 7150
 	1    0    0    -1
@@
 F 0 "U5" H 1700 4450 40  0000 L BNB
 F 1 "ATMEGA328P" H 1700 4375 40  0000 L BNN
-F 2 "SMD_Packages:PLCC-32" H 2925 1675 50  0001 C CNN
+F 2 "" H 2925 1675 50  0001 C CNN
 F 3 "" H 2400 3250 60  0001 C CNN
-F 4 "mfr_pn" H 2400 3250 60  0001 C CNN "manf#"
+F 4 "" H 2400 3250 60  0001 C CNN "manf#"
 	1    2400 3250
 	1    0    0    -1
@@
 F 0 "X2" V 750 3100 40  0000 C CNB
 F 1 "8MHz" V 1050 3125 40  0000 C CNN
-F 2 "velokey-footprints:xtal_3.2x1.5mm" H 900 3050 60  0001 C CNN
+F 2 "" H 900 3050 60  0001 C CNN
 F 3 "" H 900 3050 60  0000 C CNN
 	1    900  3050
@@
 F 0 "C22" H 1300 7150 40  0000 L CNB
 F 1 "47uF,25V" H 1250 7075 40  0000 L CNN
-F 2 "velokey-footprints:c_elec_3x5.3" H 1225 7150 60  0001 C CNN
+F 2 "" H 1225 7150 60  0001 C CNN
 F 3 "" H 1225 7150 60  0000 C CNN
-F 4 "mfr_pn" H 1225 7150 60  0001 C CNN "manf#"
+F 4 "" H 1225 7150 60  0001 C CNN "manf#"
 	1    1225 7150
 	1    0    0    -1
@@
 F 2 "" H 6150 1875 40  0001 C CNN
 F 3 "" H 6150 1875 40  0000 C CNN
-F 4 "mfr_pn" H 6150 1875 40  0001 C CNN "manf#"
+F 4 "" H 6150 1875 40  0001 C CNN "manf#"
 	1    6150 1875
 	1    0    0    -1
@@
 F 2 "" H 7825 1875 40  0001 C CNN
 F 3 "" H 7825 1875 40  0000 C CNN
-F 4 "mfr_pn" H 7825 1875 40  0001 C CNN "manf#"
+F 4 "" H 7825 1875 40  0001 C CNN "manf#"
 	1    7825 1875
 	1    0    0    -1
@@
 F 0 "C25" H 5975 2550 40  0000 L CNB
 F 1 "1uF" H 5925 2475 40  0000 L CNN
-F 2 "velokey-footprints:c_elec_3x5.3" H 5900 2550 60  0001 C CNN
+F 2 "" H 5900 2550 60  0001 C CNN
 F 3 "" H 5900 2550 60  0000 C CNN
-F 4 "mfr_pn" H 5900 2550 60  0001 C CNN "manf#"
+F 4 "" H 5900 2550 60  0001 C CNN "manf#"
 	1    5900 2550
 	1    0    0    -1
@@
 F 0 "C26" H 6475 2550 40  0000 L CNB
 F 1 "1uF" H 6425 2475 40  0000 L CNN
-F 2 "velokey-footprints:c_elec_3x5.3" H 6400 2550 60  0001 C CNN
+F 2 "" H 6400 2550 60  0001 C CNN
 F 3 "" H 6400 2550 60  0000 C CNN
-F 4 "mfr_pn" H 6400 2550 60  0001 C CNN "manf#"
+F 4 "" H 6400 2550 60  0001 C CNN "manf#"
 	1    6400 2550
 	1    0    0    -1
@@
 F 0 "C27" H 7650 2550 40  0000 L CNB
 F 1 "1uF" H 7600 2475 40  0000 L CNN
-F 2 "velokey-footprints:c_elec_3x5.3" H 7575 2550 60  0001 C CNN
+F 2 "" H 7575 2550 60  0001 C CNN
 F 3 "" H 7575 2550 60  0000 C CNN
-F 4 "mfr_pn" H 7575 2550 60  0001 C CNN "manf#"
+F 4 "" H 7575 2550 60  0001 C CNN "manf#"
 	1    7575 2550
 	1    0    0    -1
@@
 F 0 "C28" H 8150 2550 40  0000 L CNB
 F 1 "1uF" H 8100 2475 40  0000 L CNN
-F 2 "velokey-footprints:c_elec_3x5.3" H 8075 2550 60  0001 C CNN
+F 2 "" H 8075 2550 60  0001 C CNN
 F 3 "" H 8075 2550 60  0000 C CNN
-F 4 "mfr_pn" H 8075 2550 60  0001 C CNN "manf#"
+F 4 "" H 8075 2550 60  0001 C CNN "manf#"
 	1    8075 2550
 	1    0    0    -1
@@
 F 0 "R17" H 5950 2350 40  0000 C CNB
 F 1 "10k" V 5900 2250 40  0000 C CNN
-F 2 "velokey-footprints:R_0603_HandSoldering" H 5900 2250 60  0001 C CNN
+F 2 "" H 5900 2250 60  0001 C CNN
 F 3 "" H 5900 2250 60  0001 C CNN
-F 4 "mfr_pn" H 5900 2250 60  0001 C CNN "manf#"
+F 4 "" H 5900 2250 60  0001 C CNN "manf#"
 	1    5900 2250
 	1    0    0    -1
@@
 F 0 "R18" H 6450 2350 40  0000 C CNB
 F 1 "10k" V 6400 2250 40  0000 C CNN
-F 2 "velokey-footprints:R_0603_HandSoldering" H 6400 2250 60  0001 C CNN
+F 2 "" H 6400 2250 60  0001 C CNN
 F 3 "" H 6400 2250 60  0001 C CNN
-F 4 "mfr_pn" H 6400 2250 60  0001 C CNN "manf#"
+F 4 "" H 6400 2250 60  0001 C CNN "manf#"
 	1    6400 2250
 	1    0    0    -1
@@
 F 0 "R19" H 7625 2350 40  0000 C CNB
 F 1 "10k" V 7575 2250 40  0000 C CNN
-F 2 "velokey-footprints:R_0603_HandSoldering" H 7575 2250 60  0001 C CNN
+F 2 "" H 7575 2250 60  0001 C CNN
 F 3 "" H 7575 2250 60  0001 C CNN
-F 4 "mfr_pn" H 7575 2250 60  0001 C CNN "manf#"
+F 4 "" H 7575 2250 60  0001 C CNN "manf#"
 	1    7575 2250
 	1    0    0    -1
@@
 F 0 "R20" H 8125 2350 40  0000 C CNB
 F 1 "10k" V 8075 2250 40  0000 C CNN
-F 2 "velokey-footprints:R_0603_HandSoldering" H 8075 2250 60  0001 C CNN
+F 2 "" H 8075 2250 60  0001 C CNN
 F 3 "" H 8075 2250 60  0001 C CNN
-F 4 "mfr_pn" H 8075 2250 60  0001 C CNN "manf#"
+F 4 "" H 8075 2250 60  0001 C CNN "manf#"
 	1    8075 2250
 	1    0    0    -1
