File: KiCad/velokey.sch (KiCad schematic (older format))
At the start: 34 parts, among them P1 USB_micro, P2 CONN_01X13, P3 CONN_01X13, P4 CONN_01X01, P5 CONN_01X01, P6 CONN_01X01, U1 MIC5528, U2 STF202, U3 ATSAMD21E, X1 ABS07

Commit message: schematic, work in progress
Parts:
- removed C10, C8, C9: 100nF, hack-footprints:C_0603_HandSoldering, symbol C_Small
- removed C3, C4: 10uF, hack-footprints:c_elec_3x5.3, symbol CP_Small
- removed JP1: Jumper_NO_Small, hack-footprints:SMD_Jumper, symbol Jumper_NO_Small
- removed L1: BLM18EG221, hack-footprints:L_0603_HandSoldering, symbol FERRITE_BEAD
- removed L2: 10uH, hack-footprints:ELLVFG, symbol L_Small
- removed P2, P3: CONN_01X13, hack-footprints:Pin_Castellated_1x13, symbol CONN_01X13
- removed P4, P5, P6: CONN_01X01, hack-footprints:Pin_Castellated_1x01, symbol CONN_01X01
- removed U3: ATSAMD21E, hack-footprints:QFN-32-1EP_5x5mm_Pitch0.5mm, symbol ATSAMD21E
- added C? (x5): 100nF, symbol C_Small
- added C?: 10uF, symbol CP_Small
- added C?: CP_Small, symbol CP_Small
- added D? (x2): RED, hack-footprints:LED_0603_HandSoldering, symbol Led_Small
- added L?: FERRITE_BEAD, symbol FERRITE_BEAD
- added L?: L_Small, symbol L_Small
- added P?: CONN_02X5, symbol CONN_02X5
- added P?: SPI, symbol CONN_02X3
- added P?: POWER, symbol CONN_01X08
- added P?: ANALOG, symbol CONN_01X06
- added P?: DIGITAL_01, symbol CONN_01X08
- added P?: DIGITAL_02, symbol CONN_01X10
- added Q?: MMBF170, SOT-23, symbol MMBF170
- added R? (x4): 330, hack-footprints:R_0603_HandSoldering, symbol R_Small
- added U? (x2): SAMD21G18A, symbol SAMD21G18A
- R4: value 330 -> 39
Connections:
- net labels added: 3V3, 5V, A0, A1, A2, A3, A4, A5, AREF, BLINK, D0, D1, D2, D3, D4, D5, D6, D7, D8, D9, DBG_MISO, DBG_MOSI, DBG_SCK, D_N, D_P, MISO, MOSI, RESET, RST, RXD, RX_LED, SCK, SCL, SDA, SS, SWCLK, SWDIO, TXD, TX_LED, USB_HOST_EN, USB_N, USB_P, VIN
- net labels removed: !RESET, PA02/A0, PA03/A1, PA04/A2, PA05/A3, PA06/A4, PA07/A5, PA08/0, PA09/1, PA10/2, PA11/3, PA14/4, PA15/5, PA16/6, PA17/7, PA18/8, PA19/9, PA22/10, PA23/11, PA27/12, PA28/13, PA30/SWCLK, PA31/SWDIO, USB-D+, USB-D-, VDD, VDDANA, VDDCORE, VDDF, VLDO
- wire segments 86 -> 153
- no-connect marks 4 -> 8
Other:
- note added: "INTERFACES"
- note removed: "BREAKOUT PINS + CASTELLATED EDGES"
- note removed: "JUMPER"
- moved on the sheet: C11, D1, FID1, FID2, FID3, R2, R3, R4, S1

Commit message: schematic, work in progress
Parts:
- removed U1: MIC5528, hack-footprints:DFN-6-1EP_1.2x1.2mm_Pitch0.4mm, symbol MIC5528
- added C?: 100nF, symbol C_Small
- added C?: 10uF, symbol CP_Small
- added C?: 1uF, hack-footprints:C_0603_HandSoldering, symbol C_Small
- added C?: 10uF, hack-footprints:C_0603_HandSoldering, symbol C_Small
- added D?: MBR120, symbol Led_Schottky
- added D?: LED_CHG, hack-footprints:LED_0603_HandSoldering, symbol Led_Small
- added P?: JSTPH, symbol CONN_01X02
- added P?: LCD_DISPLAY, symbol CONN_01X10
- added P?: Bluefruit, symbol CONN_01X08
- added R?: 100k, hack-footprints:R_0603_HandSoldering, symbol R_Small
- added R?: 330, hack-footprints:R_0603_HandSoldering, symbol R_Small
- added R?: 10k, hack-footprints:R_0603_HandSoldering, symbol R_Small
- added U?: SPX3819-3V3, symbol SPX3819-3V3
- added U?: MCP73831, symbol MCP73831
- C1, C2: value 2.2uF -> 10uF
- C6, C7: value 10pF -> 22pF
- D1: value RED -> LED_BLINK
- D?: value RED -> LED_RX
- D?: value RED -> LED_TX
- P?: value CONN_02X5 -> SWD
Connections:
- net DBG_MISO is gone; now on net MISO: P?.1 (P1), P?.4 (P4), U?.21 (PA12/I2C/EIC/SCOM2PAD0+/TC2)
- net DBG_MOSI is gone; now on net MOSI: U?.19 (PB10/EIC/SCOM4PAD2/TC5)
- net DBG_SCK is gone; now on net SCK: P?.3 (P3), U?.20 (PB11/EIC/SCOM4PAD3/TC5)
- net AREF: now also C?.1, C?.1
- net D2: now also U?.23 (PA14/XIN/EIC/SCOM2PAD2+/TC3); no longer U?.13 (PA8/I2C/AIN16/SCOM2PAD0+/TC0)
- net D4: no longer U?.23 (PA14/XIN/EIC/SCOM2PAD2+/TC3)
- net D5: no longer U?.24 (PA15/XOUT/EIC/SCOM2PAD3+/TC3)
- net D8: no longer U?.11 (PA6/EIC/AIN6/SCOM0PAD2/TC1)
- net D9: no longer U?.12 (PA7/EIC/AIN7/SCOM0PAD3/TC1)
- net GND: now also C?.2, C?.2, C?.2, C?.2, P?.1 (P1), P?.2 (P2), P?.2 (P2), R?.1, U?.2 (GND), U?.2 (VSS)
- net MISO: no longer U?.28 (PA19/EIC/SCOM1PAD3+/TC3)
- net MOSI: no longer U?.25 (PA16/I2C/EIC/SCOM1PAD0+/TC2)
- net SCK: no longer U?.26 (PA17/I2C/EIC/SCOM1PAD1+/TC2)
- net SS: no longer U?.27 (PA18/EIC/SCOM1PAD2+/TC3)
- net VBUS: now also D?.1 (A), D?.2 (K), R?.2, U?.1 (VIN), U?.4 (VIN)
- net VIN: now also P?.4 (P4)
- net 3V3 renamed +3V3
- net +3V3: now also C?.1, P?.2 (P2), P?.8 (P8), U?.5 (VOUT)
- net BLINK renamed D13
- net D13: no longer U?.22 (PA13/I2C/EIC/SCOM2PAD1+/TC2)
- new net: R?.1, U?.3 (EN)
- new net: R?.1, U?.1 (STAT)
- new net: R?.2, U?.5 (PROG)
- new net: D?.2 (K), R?.2
- new net CS_CARD: P?.5 (P5)
- new net CS_LCD: P?.6 (P6), U?.27 (PA18/EIC/SCOM1PAD2+/TC3)
- new net D/C: P?.4 (P4), U?.11 (PA6/EIC/AIN6/SCOM0PAD2/TC1)
- new net D12: U?.28 (PA19/EIC/SCOM1PAD3+/TC3)
- new net DSR: P?.3 (P3)
- new net DTR: P?.7 (P7)
- new net MISO_LCD: P?.7 (P7), U?.25 (PA16/I2C/EIC/SCOM1PAD0+/TC2)
- new net PWM_LCD: P?.9 (P9)
- new net RST_LCD: P?.3 (P3), U?.12 (PA7/EIC/AIN7/SCOM0PAD3/TC1)
- new net RX_BT: P?.6 (P6), U?.24 (PA15/XOUT/EIC/SCOM2PAD3+/TC3)
- new net SCK_LCD: P?.8 (P8), U?.26 (PA17/I2C/EIC/SCOM1PAD1+/TC2)
- new net STS: P?.1 (P1)
- new net TX_BT: P?.5 (P5), U?.13 (PA8/I2C/AIN16/SCOM2PAD0+/TC0)
- new net VBAT: C?.1, D?.1 (A), P?.1 (P1), U?.3 (VBAT)
- no-connect marks 8 -> 15
Other:
- note added: "10k = 100mA\n5.0k = 200mA\n2.0k = 500mA\n1.0k = 1000mA"
- note added: "32.768kHz"
- note added: "INDICATORS"
- note added: "LDO VOLTAGE REGULATOR"
- note added: "LIPO CHARGER"
- note added: "MICRO CONTROLLER POWER"
- note added: "where do CS_CARD and\nPWM_LCD connect ?"
- note removed: "V_REG"
- moved on the sheet: C1, C11, C2, C5, C6, C7, C?, D1, D?, L?, P1, P?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

Commit message: schematic, work in progress
Parts:
- R5: renamed from R?; value 10k -> 2k
- gave numbers to parts that had none: 36
- renumbered C7 to C10, C5 to C3, C11 to C4, C1 to C6, C2 to C7, C6 to C9, D1 to D3, R3 to R1, R1 to R2, R2 to R8, U2 to U1
Connections:
- net D12 is gone; now on net PWM_LCD: U2.28 (PA19/EIC/SCOM1PAD3+/TC3)
- net D4 is gone; now on net TX_BT: P9.5 (P5)
- net D5 is gone; now on net RX_BT: P9.6 (P6)
- net D8 is gone; now on net D/C: P7.1 (P1)
- net D9 is gone; now on net RST_LCD: P7.2 (P2)
- net SS is gone; now on net CS_LCD: P7.3 (P3)
- net VBAT is gone; now on net +BATT: C5.1, D2.1 (A), P3.1 (P1), U3.3 (VBAT)
- net VIN: no longer P4.4 (P4)
- net D0 renamed ENC_RXD
- net D1 renamed ENC_TXD
- new net VIN_BT: P4.4 (P4)
- no-connect marks 15 -> 17
Other:
- note added: "D0"
- note added: "D1"
- note added: "D10"
- note added: "D11"
- note added: "D12"
- note added: "D13"
- note added: "D4"
- note added: "D5"
- note added: "D8"
- note added: "D9"

Commit message: schematic, work in progress
Connections:
- net D13 is gone; now on net SCK_LCD: Q1.1 (G), R11.2
Other:
- moved on the sheet: D4, D5, R10, R9
Changed lines of the file:
@@
 LIBS:velokey
 LIBS:power
-LIBS:PiPower_sch
-LIBS:arthurc
 LIBS:velokey-cache
 EELAYER 25 0
@@
 L Led_Small D4
 U 1 1 56A6A71E
-P 6825 5575
-F 0 "D4" V 6825 5525 40  0000 R CNB
-F 1 "LED_RX" V 6750 5525 40  0000 R CNN
-F 2 "hack-footprints:LED_0603_HandSoldering" V 6825 5575 40  0001 C CNB
-F 3 "https://github.com/MickMad/HACK/tree/master/kicad/datasheets/S_110_LTST-C190KRKT.pdf" V 6825 5575 40  0001 C CNB
-F 4 "LTST-C190KRKT" V 6825 5575 60  0001 C CNN "manf#"
-	1    6825 5575
+P 6900 5575
+F 0 "D4" V 6900 5525 40  0000 R CNB
+F 1 "LED_RX" V 6825 5525 40  0000 R CNN
+F 2 "hack-footprints:LED_0603_HandSoldering" V 6900 5575 40  0001 C CNB
+F 3 "https://github.com/MickMad/HACK/tree/master/kicad/datasheets/S_110_LTST-C190KRKT.pdf" V 6900 5575 40  0001 C CNB
+F 4 "LTST-C190KRKT" V 6900 5575 60  0001 C CNN "manf#"
+	1    6900 5575
 	0    -1   -1   0
 $EndComp
@@
 L R_Small R9
 U 1 1 56A6A725
-P 6825 5350
-F 0 "R9" H 6875 5350 40  0000 L CNB
-F 1 "330" V 6825 5350 40  0000 C CNN
-F 2 "hack-footprints:R_0603_HandSoldering" H 6825 5350 40  0001 C CNB
-F 3 "https://github.com/MickMad/HACK/tree/master/kicad/datasheets/0011330P1.pdf" H 6825 5350 40  0001 C CNB
-F 4 "RC0603FR-07330RL" H 6825 5350 60  0001 C CNN "manf#"
-	1    6825 5350
-	1    0    0    -1
-$EndComp
-Text Label 6825 5150 0    40   ~ 8
+P 6900 5350
+F 0 "R9" H 6950 5350 40  0000 L CNB
+F 1 "330" V 6900 5350 40  0000 C CNN
+F 2 "hack-footprints:R_0603_HandSoldering" H 6900 5350 40  0001 C CNB
+F 3 "https://github.com/MickMad/HACK/tree/master/kicad/datasheets/0011330P1.pdf" H 6900 5350 40  0001 C CNB
+F 4 "RC0603FR-07330RL" H 6900 5350 60  0001 C CNN "manf#"
+	1    6900 5350
+	1    0    0    -1
+$EndComp
+Text Label 6900 5150 0    40   ~ 8
 3V3
 $Comp
 L Led_Small D5
 U 1 1 56A6A918
-P 7225 5575
-F 0 "D5" V 7225 5525 40  0000 R CNB
-F 1 "LED_TX" V 7150 5525 40  0000 R CNN
-F 2 "hack-footprints:LED_0603_HandSoldering" V 7225 5575 40  0001 C CNB
-F 3 "https://github.com/MickMad/HACK/tree/master/kicad/datasheets/S_110_LTST-C190KRKT.pdf" V 7225 5575 40  0001 C CNB
-F 4 "LTST-C190KRKT" V 7225 5575 60  0001 C CNN "manf#"
-	1    7225 5575
+P 7275 5575
+F 0 "D5" V 7275 5525 40  0000 R CNB
+F 1 "LED_TX" V 7200 5525 40  0000 R CNN
+F 2 "hack-footprints:LED_0603_HandSoldering" V 7275 5575 40  0001 C CNB
+F 3 "https://github.com/MickMad/HACK/tree/master/kicad/datasheets/S_110_LTST-C190KRKT.pdf" V 7275 5575 40  0001 C CNB
+F 4 "LTST-C190KRKT" V 7275 5575 60  0001 C CNN "manf#"
+	1    7275 5575
 	0    -1   -1   0
 $EndComp
@@
 L R_Small R10
 U 1 1 56A6A91F
-P 7225 5350
-F 0 "R10" H 7275 5350 40  0000 L CNB
-F 1 "330" V 7225 5350 40  0000 C CNN
-F 2 "hack-footprints:R_0603_HandSoldering" H 7225 5350 40  0001 C CNB
-F 3 "https://github.com/MickMad/HACK/tree/master/kicad/datasheets/0011330P1.pdf" H 7225 5350 40  0001 C CNB
-F 4 "RC0603FR-07330RL" H 7225 5350 60  0001 C CNN "manf#"
-	1    7225 5350
-	1    0    0    -1
-$EndComp
-Text Label 7225 5150 0    40   ~ 8
+P 7275 5350
+F 0 "R10" H 7325 5350 40  0000 L CNB
+F 1 "330" V 7275 5350 40  0000 C CNN
+F 2 "hack-footprints:R_0603_HandSoldering" H 7275 5350 40  0001 C CNB
+F 3 "https://github.com/MickMad/HACK/tree/master/kicad/datasheets/0011330P1.pdf" H 7275 5350 40  0001 C CNB
+F 4 "RC0603FR-07330RL" H 7275 5350 60  0001 C CNN "manf#"
+	1    7275 5350
+	1    0    0    -1
+$EndComp
+Text Label 7275 5150 0    40   ~ 8
 3V3
-Text Label 6825 5975 0    40   ~ 8
+Text Label 6900 5975 0    40   ~ 8
 RX_LED
-Text Label 7225 5975 0    40   ~ 8
+Text Label 7275 5975 0    40   ~ 8
 TX_LED
 $Comp
@@
 32.768kHz
 NoConn ~ 4475 2975
-Text Label 6550 5975 0    40   ~ 8
-D13
 $Comp
 L SPX3819-3V3 U4
@@
 	6475 5975 6550 5975
 Wire Wire Line
-	6825 5450 6825 5475
-Wire Wire Line
-	6825 5250 6825 5150
-Wire Wire Line
-	6825 5675 6825 5975
-Wire Wire Line
-	7225 5450 7225 5475
-Wire Wire Line
-	7225 5250 7225 5150
-Wire Wire Line
-	7225 5675 7225 5975
+	6900 5450 6900 5475
+Wire Wire Line
+	6900 5250 6900 5150
+Wire Wire Line
+	6900 5675 6900 5975
+Wire Wire Line
+	7275 5450 7275 5475
+Wire Wire Line
+	7275 5250 7275 5150
+Wire Wire Line
+	7275 5675 7275 5975
 Wire Wire Line
 	6500 6050 6500 5975
@@
 Text Label 7475 2875 0    40   ~ 8
 PWM_LCD
+Text Label 6550 5975 0    40   ~ 8
+SCK_LCD
 $EndSCHEMATC
