File: KiCad/velokey.sch (KiCad schematic (older format))
At the start: 56 parts, among them P1 USB_micro, P10 ANALOG, P2 LCD_DISPLAY, P3 JSTPH, P4 Bluefruit, P5 SPI, P6 SWD, P7 DIGITAL_02, P8 POWER, P9 DIGITAL_01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

Commit message: work in progress
Parts:
- C10, C3, C4, C5, C6, C7, C8, C9: footprint hack-footprints:C_0603_HandSoldering -> velokey-footprints:C_0603_HandSoldering
- D1, D3, D4, D5: footprint hack-footprints:LED_0603_HandSoldering -> velokey-footprints:LED_0603_HandSoldering
- FID1, FID2, FID3: footprint hack-footprints:FIDUCIAL -> velokey-footprints:FIDUCIAL
- LOGO1: footprint hack-footprints:OSHW-LOGO -> velokey-footprints:OSHW-LOGO
- P1: footprint hack-footprints:ST-USB-001G -> velokey-footprints:ST-USB-001G
- R1, R10, R11, R2, R3, R4, R5, R6, R7, R8, R9: footprint hack-footprints:R_0603_HandSoldering -> velokey-footprints:R_0603_HandSoldering
- S1: footprint hack-footprints:SPST-PTS_810 -> velokey-footprints:SPST-PTS_810
- U1: footprint hack-footprints:TSOP-6 -> velokey-footprints:TSOP-6
- X1: footprint hack-footprints:xtal_3.2x1.5mm -> velokey-footprints:xtal_3.2x1.5mm

Commit message: added OTS schematic
Parts:
- C10, C9: footprint velokey-footprints:C_0603_HandSoldering -> (none); manf# CC0603JRNPO9BN100 -> (none)
- C3: footprint velokey-footprints:C_0603_HandSoldering -> (none); manf# CC0603KRX7R9BB472 -> (none)
- C4: footprint velokey-footprints:C_0603_HandSoldering -> (none); manf# CC0603KRX7R9BB104 -> (none)
- C5, C6, C7, C8: footprint velokey-footprints:C_0603_HandSoldering -> (none); manf# CC0603MRX5R5BB225 -> (none)
- D1, D3, D4, D5: footprint velokey-footprints:LED_0603_HandSoldering -> (none); manf# LTST-C190KRKT -> (none)
- FID1, FID2, FID3: footprint velokey-footprints:FIDUCIAL -> (none)
- L1: manf# BLM18EG221SN1D -> (none)
- L2: manf# ELL-VFG100MC -> (none)
- LOGO1: footprint velokey-footprints:OSHW-LOGO -> (none)
- P1: footprint velokey-footprints:ST-USB-001G -> (none); manf# 10118193-0001LF -> (none)
- Q1: footprint SOT-23 -> (none)
- R1: footprint velokey-footprints:R_0603_HandSoldering -> (none); manf# RC0603FR-0710KL -> (none)
- R10, R11, R3, R4, R5, R6, R8, R9: footprint velokey-footprints:R_0603_HandSoldering -> (none); manf# RC0603FR-07330RL -> (none)
- R2, R7: footprint velokey-footprints:R_0603_HandSoldering -> (none); manf# RC0603FR-071ML -> (none)
- S1: footprint velokey-footprints:SPST-PTS_810 -> (none); manf# PTS810 SJM 250 SMTR LFS -> (none)
- U1: footprint velokey-footprints:TSOP-6 -> (none); manf# STF202-22T1G -> (none)
- U2: manf# SAMD21G18A-AUT -> (none)
- U4: manf# SPX3819M5-L-3-3 -> (none)
- X1: footprint velokey-footprints:xtal_3.2x1.5mm -> (none); manf# ABS07-32.768KHZ-7-T -> (none)
