File: KiCad/OTS.kicad_pcb (KiCad board)
At the start: 2 copper layers, 134.6 x 52.1 mm, 26 parts, among them P43 POWER_UP, U10 ProMini, U7 EZbluefruit, U8 LCD_TFT, U9 FeatherM0

Commit message: added L2 and LITE connections
Connections:
- net GND renamed /GND
- net Net-(C32-Pad1) renamed /POWERUP
- R21 pad 1: /VELO/VCC -> /VCC
- R22 pad 1: /VELO/VCC -> /VCC
- R23 pad 1: /VELO/VCC -> /VCC
- R24 pad 1: /VELO/VCC -> /VCC
- R25 pad 1: /VELO/VCC -> /VCC
- R26 pad 1: /VELO/VCC -> /VCC
- R27 pad 1: /VELO/VCC -> /VCC
- U10 pad 9: /VELO/VCC -> /VCC
- U7 pad 5: Net-(U7-Pad5) -> /L2
- U7 pad 9: /VELO/VCC -> /VCC
- U8 pad 1: /VELO/VCC -> /LITE
- U8 pad 9: /VELO/VCC -> /VCC
- U9 pad 14: /VELO/VCC -> /VCC
- U9 pad 20: Net-(U9-Pad20) -> /LITE
- U9 pad 21: Net-(U9-Pad21) -> /L2
Routing:
- net /VELO/VCC: track 389.1 -> 0.00 mm, vias 1 -> 0
- net /VCC: track 0.00 -> 309.5 mm, vias 0 -> 1
- net /LITE: track 0.00 -> 50.0 mm, vias 0 -> 1
- net /L2: track 0.00 -> 49.0 mm, vias 0 -> 2
- net /GND: track 356.6 -> 376.1 mm
- net Net-(U9-Pad21): track 2.54 -> 0.00 mm
- net Net-(U9-Pad20): track 2.54 -> 0.00 mm
- net Net-(U7-Pad5): track 2.54 -> 0.00 mm
- net Net-(U7-Pad1): track 78.0 -> 78.6 mm

Commit message: Git issue #1,#2,#5,#7 closed
Connections:
- U9 pad 16: Net-(U9-Pad16) -> /GND
- U9 pad 28: /GND -> Net-(U9-Pad28)
Routing:
- net /GND: track 376.1 -> 322.6 mm
- net /VCC: track 309.5 -> 267.8 mm
- net Net-(U9-Pad28): track 0.00 -> 2.54 mm
- net Net-(U9-Pad16): track 2.54 -> 0.00 mm
- net /L2: track 49.0 -> 50.9 mm
