File: kicad/OTS_2/OTS2_encA.kicad_pcb (KiCad board)
At the start: 2 copper layers, 35.6 x 35.6 mm, 11 parts

Commit message: encoder daughter boards, WIP
Changed lines of the file:
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@@
-(kicad_pcb (version 4) (host pcbnew 4.1.0-alpha+201607210716+6990~46~ubuntu15.10.1-product)
+(kicad_pcb (version 20160815) (host pcbnew 4.1.0-alpha+201609021633+7109~49~ubuntu16.04.1-product)
   (general
     (links 19)
@@
     (uvia_dia 0.3)
     (uvia_drill 0.1)
+    (diff_pair_gap 0.25)
+    (diff_pair_width 0.2)
   )
   (net_class 20mil ""
@@
     (uvia_dia 0.3)
     (uvia_drill 0.1)
+    (diff_pair_gap 0.25)
+    (diff_pair_width 0.2)
     (add_net /eEAA)
     (add_net /eEAB)
@@
     (uvia_dia 0.3)
     (uvia_drill 0.1)
+    (diff_pair_gap 0.25)
+    (diff_pair_width 0.2)
     (add_net /eGND)
     (add_net /eVCC)
@@
     (uvia_dia 0.3)
     (uvia_drill 0.1)
+    (diff_pair_gap 0.25)
+    (diff_pair_width 0.2)
   )
   (module velokey-footprints:R_1210_HandSoldering (layer B.Cu)
@@
     (descr "Through hole pin header")
     (tags "pin header")
-    (fp_text reference eP8 (at 0 -5.1) (layer F.SilkS)
-      (effects (font (size 1 1) (thickness 0.15)))
+    (fp_text reference eP8 (at 0 -2.54) (layer B.SilkS)
+      (effects (font (size 1 1) (thickness 0.15)) (justify mirror))
     )
     (fp_text value ENC_A_4 (at 0 -3.1) (layer F.Fab) hide
@@
     (descr "Through hole pin header")
     (tags "pin header")
-    (fp_text reference eP6 (at 0 -5.1) (layer F.SilkS)
-      (effects (font (size 1 1) (thickness 0.15)))
+    (fp_text reference eP6 (at 0 -2.54) (layer B.SilkS)
+      (effects (font (size 1 1) (thickness 0.15)) (justify mirror))
     )
     (fp_text value ENC_A_2 (at 0 -3.1) (layer F.Fab) hide
@@
     (descr "Through hole pin header")
     (tags "pin header")
-    (fp_text reference eP5 (at 0 -5.1 90) (layer F.SilkS)
-      (effects (font (size 1 1) (thickness 0.15)))
+    (fp_text reference eP5 (at 2.54 1.27 360) (layer B.SilkS)
+      (effects (font (size 1 1) (thickness 0.15)) (justify mirror))
     )
     (fp_text value ENC_A_1 (at 0 -3.1 90) (layer F.Fab) hide
@@
     (descr "Through hole pin header")
     (tags "pin header")
-    (fp_text reference eP7 (at 0 -5.1 90) (layer F.SilkS)
-      (effects (font (size 1 1) (thickness 0.15)))
+    (fp_text reference eP7 (at -2.54 1.27 360) (layer B.SilkS)
+      (effects (font (size 1 1) (thickness 0.15)) (justify mirror))
     )
     (fp_text value ENC_A_3 (at 0 -3.1 90) (layer F.Fab) hide
@@
   (module velokey-footprints:TSWA3NCD23LFS (layer F.Cu)
     (at 42.545 40.64 270)
-    (fp_text reference eE3 (at 1.905 0) (layer F.SilkS)
-      (effects (font (size 1 1) (thickness 0.15)))
-    )
-    (fp_text value ENC_A (at -1.905 0 180) (layer F.Fab)
-      (effects (font (size 1 1) (thickness 0.15)))
+    (fp_text reference eE3 (at 1.905 0 540) (layer B.SilkS)
+      (effects (font (size 1 1) (thickness 0.15)) (justify mirror))
+    )
+    (fp_text value ENC_A (at -1.905 0 180) (layer B.SilkS)
+      (effects (font (size 1 1) (thickness 0.15)) (justify mirror))
     )
     (fp_circle (center 0 0) (end 10 0) (layer F.SilkS) (width 0.1016))

Commit message: gerbers for encA, encB, encC, main - ready
Parts:
- moved eP8 59.1 mm to (29.8, 98.4), turned to 180 degrees
- moved eC29 50.8 mm to (47.0, 98.4)
- moved eC30 50.8 mm to (34.3, 98.4)
- moved eC31 50.8 mm to (38.1, 98.4)
- moved eE3 50.8 mm to (42.5, 91.4)
- moved eP5 50.8 mm to (41.3, 78.7)
- moved eP7 50.8 mm to (41.3, 104.1)
- moved eR21 50.8 mm to (47.0, 84.5)
- moved eR22 50.8 mm to (34.3, 84.5)
- moved eR23 50.8 mm to (38.1, 84.5)
- moved eP6 49.5 mm to (29.8, 84.5)
Routing:
- net /eEAB: track 27.0 -> 41.6 mm, vias 1 -> 0
- net /eGND: track 55.8 -> 43.0 mm
- net /eEAA: track 35.4 -> 28.9 mm
- net /eVCC: track 31.3 -> 26.6 mm, vias 3 -> 1
- net /eEAS: track 30.7 -> 33.7 mm, vias 0 -> 1
- added copper zone on B.Cu, net /eGND
- added copper zone on F.Cu, net /eVCC
