File: kicad/OTS_2/OTS2_encB.kicad_pcb (KiCad board)
At the start: 2 copper layers, 35.6 x 35.6 mm, 11 parts

Commit message: gerbers for encA, encB, encC, main - ready
Parts:
- moved eP10 60.1 mm to (154.3, 98.4)
- moved eC33 50.8 mm to (137.2, 84.5)
- moved eC34 50.8 mm to (149.9, 84.5)
- moved eC35 50.8 mm to (146.1, 84.5)
- moved eE4 50.8 mm to (141.6, 91.4)
- moved eP11 50.8 mm to (140.3, 104.1)
- moved eP9 50.8 mm to (142.9, 78.7)
- moved eR25 50.8 mm to (137.2, 98.4)
- moved eR26 50.8 mm to (149.9, 98.4)
- moved eR27 50.8 mm to (146.1, 98.4)
- moved eP12 42.5 mm to (154.3, 84.5), turned to 0 degrees
Routing:
- net /eEBS: track 19.1 -> 47.5 mm
- net /eEBA: track 33.9 -> 29.6 mm
- net /eVCC: track 66.9 -> 65.3 mm
- added copper zone on B.Cu, net /eGND
- added copper zone on F.Cu, net /eVCC
