File: kicad/OTS_2/OTS2_main.kicad_pcb (KiCad board)
At the start: 2 copper layers, 134.6 x 73.7 mm, 60 parts, among them J1 LCD_Lite, P1 ENC_C_1, P10 ENC_B_2, P11 ENC_B_3, P12 ENC_B_4, P13 ENC_C_4, P2 ENC_C_2, P3 ENC_C_3, P4 ENC_C_4, P5 ENC_A_1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

Commit message: gerbers for encA, encB, encC, main - ready
Parts:
- moved P6 21.1 mm to (29.8, 33.7)
- moved P10 21.1 mm to (154.3, 47.6)
- moved P8 8.26 mm to (29.8, 47.6), turned to 180 degrees
- moved P12 8.25 mm to (154.3, 33.7), turned to 0 degrees
- moved P11 2.54 mm to (142.9, 53.3), turned to 270 degrees
Routing:
- net /VCC: track 498.5 -> 518.1 mm
- net /EBS: track 82.8 -> 95.2 mm
- net /EAA: track 68.5 -> 80.2 mm
- net /GND: track 461.5 -> 467.9 mm
- net /EBA: track 112.6 -> 108.4 mm
